File: polarshield3.0b.sch (EAGLE design)
At the start: 45 parts

Commit message: Minor changes based on first board.
Parts:
- removed M1_CONN, M2_CONN: (no value), pinhead:PINHD-1X4/90
- added X1, X4: (no value), con-molex-micro-fit-3_0:HEADER_POS4_43045-0401
- added X5, X6: (no value), con-molex-micro-fit-3_0:HEADER_POS6_43045-0600
Connections:
- removed net N$20: M2_CONN.1, MOTOR_2.2B
- removed net N$21: M2_CONN.2, MOTOR_2.2A
- removed net N$22: M2_CONN.3, MOTOR_2.1A
- removed net N$23: M2_CONN.4, MOTOR_2.1B
- new net N$24: MOTOR_2.1B, X4.4
- new net N$25: MOTOR_2.2B, X4.1
- new net N$26: MOTOR_2.2A, X4.2
- new net N$27: MOTOR_2.1A, X4.3
- net +3V3: now also X5.4, X6.4
- net +5V: now also X5.5, X6.5
- net ENC1_A: now also X5.1
- net ENC1_B: now also X5.2
- net ENC2_A: now also X6.1
- net ENC2_B: now also X6.2
- net GND: now also X5.6, X6.6
- net GP_2: now also X5.3
- net GP_3: now also X6.3
- net N$10: now also X1.1; no longer M1_CONN.1
- net N$11: now also X1.2; no longer M1_CONN.2
- net N$12: now also X1.3; no longer M1_CONN.3
- net N$13: now also X1.4; no longer M1_CONN.4
