File: polarshield3.0c.sch (EAGLE design)
At the start: 45 parts

Commit message: Minor changes based on first board.
Parts:
- removed ISOLATE_EXT, T_IRQ_LINK: (no value), SparkFun-Connectors:M02PTH
- removed R10, R3, R6, R7: 1k, resistor:R-EU_M0805
- removed SJ7: (no value), SparkFun-Retired:SOLDERJUMPER_2WAYPASTE1&2
- added Q4, Q5, Q6, Q7: BSS138, SparkFun:MOSFET-NCHANNELSMD
- added RN1, RN2: 10k, resistor-dil:4R-NEXB38V
- added RN3: 1k, resistor-dil:4R-NEXB38V
- added SJ8: T_IRQ_LINK, SparkFun-Retired:SOLDERJUMPERNO
Connections:
- removed net N$28: SJ7.2, SPARE_BREAKOUT.4
- new net ENC1_A_HV: Q7.D, RN2D.1, SPARE_BREAKOUT.12
- new net ENC1_B_HV: Q6.D, RN2B.1, SPARE_BREAKOUT.10
- new net ENC2_A_HV: Q5.D, RN1D.1, SPARE_BREAKOUT.8
- new net ENC2_B_HV: Q4.D, RN1B.1, SPARE_BREAKOUT.6
- new net GP_1_HV: SPARE_BREAKOUT.11
- new net GP_2_HV: SPARE_BREAKOUT.9
- new net GP_3_HV: SPARE_BREAKOUT.7
- net +3V3: now also Q4.G, Q5.G, Q6.G, Q7.G, RN1A.2, RN1C.2, RN2A.2, RN2C.2; no longer SJ7.3
- net +5V: now also RN1B.2, RN1D.2, RN2B.2, RN2D.2, SPARE_BREAKOUT.4; no longer SJ7.1
- net ENC1_A: now also Q7.S, RN2C.1; no longer SPARE_BREAKOUT.12
- net ENC1_B: now also Q6.S, RN2A.1; no longer SPARE_BREAKOUT.10
- net ENC2_A: now also Q5.S, RN1C.1; no longer SPARE_BREAKOUT.8
- net ENC2_B: now also Q4.S, RN1A.1; no longer SPARE_BREAKOUT.6
- net GP_1: no longer SPARE_BREAKOUT.11
- net GP_2: no longer SPARE_BREAKOUT.9
- net GP_3: no longer SPARE_BREAKOUT.7
- net M1_STEP: now also RN3D.1; no longer R3.2
- net M2_STEP: now also RN3A.1; no longer R10.2
- net N$1: now also SJ8.2; no longer T_IRQ_LINK.2
- net N$14: now also RN3C.2; no longer R6.1
- net N$15: now also RN3B.2; no longer R7.1
- net N$19: now also RN3A.2; no longer R10.1
- net N$6: now also RN3D.2; no longer R3.1
- net N$7: no longer ISOLATE_EXT.1, ISOLATE_EXT.2
- net RX: now also RN3B.1; no longer R7.2
- net TX: now also RN3C.1; no longer R6.2
- net T_IRQ: now also SJ8.1; no longer T_IRQ_LINK.1
