File: polarshield3.0e.sch (EAGLE design)
At the start: 45 parts

Commit message: Minor changes based on first board.
Parts:
- removed ISOLATE_EXT, T_IRQ_LINK: (no value), SparkFun-Connectors:M02PTH
- removed M1_STEP, M2_STEP: (no value), polargraph3:LEDCHIPLED_0805
- removed R10, R3, R6, R7: 1k, resistor:R-EU_M0805
- removed SJ7: (no value), SparkFun-Retired:SOLDERJUMPER_2WAYPASTE1&2
- removed SPARE_BREAKOUT: (no value), pinhead:PINHD-2X6
- added CN1, CN2: DIP-BLACK-FEMALE-HEADER-VERT(8P-2.54), Seeed-Connector:DIP-BLACK-FEMALE-HEADER-VERT(8P-2.54)
- added Q4, Q5, Q6, Q7: BSS138, SparkFun:MOSFET-NCHANNELSMD
- added RN1, RN2: 10k, resistor-dil:4R-NEXB38V
- added RN3: 1k, resistor-dil:4R-NEXB38V
- added SJ8: T_IRQ_LINK, SparkFun-Retired:SOLDERJUMPERNO
Connections:
- removed net N$19: M2_STEP.A, R10.1
- removed net N$28: SJ7.2, SPARE_BREAKOUT.4
- removed net N$6: M1_STEP.A, R3.1
- new net ENC1_A_HV: CN2.1, Q7.D, RN2D.1
- new net ENC1_B_HV: CN2.2, Q6.D, RN2B.1
- new net ENC2_A_HV: CN2.5, Q5.D, RN1D.1
- new net ENC2_B_HV: CN2.6, Q4.D, RN1B.1
- net +3V3: now also CN1.3, CN1.7, Q4.G, Q5.G, Q6.G, Q7.G, RN1A.2, RN1C.2, RN2A.2, RN2C.2; no longer SJ7.3, SPARE_BREAKOUT.3
- net +5V: now also CN2.3, CN2.7, RN1B.2, RN1D.2, RN2B.2, RN2D.2; no longer SJ7.1, SPARE_BREAKOUT.5
- net ENC1_A: now also Q7.S, RN2C.1; no longer SPARE_BREAKOUT.12
- net ENC1_B: now also Q6.S, RN2A.1; no longer SPARE_BREAKOUT.10
- net ENC2_A: now also Q5.S, RN1C.1; no longer SPARE_BREAKOUT.8
- net ENC2_B: now also Q4.S, RN1A.1; no longer SPARE_BREAKOUT.6
- net GND: now also CN1.4, CN1.8, CN2.4, CN2.8; no longer M1_STEP.C, M2_STEP.C, SPARE_BREAKOUT.1, SPARE_BREAKOUT.2
- net GP_1: now also CN1.2; no longer SPARE_BREAKOUT.11
- net GP_2: now also CN1.6; no longer SPARE_BREAKOUT.9
- net GP_3: no longer SPARE_BREAKOUT.7
- net M1_STEP: no longer R3.2
- net M2_STEP: no longer R10.2
- net N$1: now also SJ8.2; no longer T_IRQ_LINK.2
- net N$14: now also RN3C.2; no longer R6.1
- net N$15: now also RN3B.2; no longer R7.1
- net N$7: no longer ISOLATE_EXT.1, ISOLATE_EXT.2
- net RX: now also RN3B.1; no longer R7.2
- net TX: now also RN3C.1; no longer R6.2
- net T_IRQ: now also SJ8.1; no longer T_IRQ_LINK.1
