File: polarshield3.0f.sch (EAGLE design)
At the start: 43 parts, among them CN1 DIP-BLACK-FEMALE-HEADER-VERT(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, CN2 DIP-BLACK-FEMALE-HEADER-VERT(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, Q4 BSS138, Q5 BSS138, Q6 BSS138, Q7 BSS138

Commit message: Added part number GF1A-E3/67A to D1, #1
Parts:
- D1: value (none) -> GF1A-E3/67A
Changed lines of the file:
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@@
 <part name="RX" library="polargraph3" deviceset="LED" device="CHIPLED_0805"/>
 <part name="+3V7" library="supply1" deviceset="+3V3" device=""/>
-<part name="D1" library="diode" deviceset="DIODE-" device="DO214BA"/>
+<part name="D1" library="diode" deviceset="DIODE-" device="DO214BA" value="GF1A-E3/67A "/>
 <part name="P+4" library="supply1" deviceset="+5V" device=""/>
 <part name="+3V8" library="supply1" deviceset="+3V3" device=""/>

Commit message: v3.0f. Removed 1k resistors, moved motor connectors and pads for mini-360.
Parts:
- U$3: value MINI-360-MP2307 -> MINI-360-MP2307MINI-360-MP2307_T; device polargraph3:MINI-360-MP2307 -> polargraph3:MINI-360-MP2307MINI-360-MP2307_T
Changed lines of the file:
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@@
 <part name="C3" library="resistor" deviceset="C-EU" device="C0805" value="100nF"/>
 <part name="C4" library="resistor" deviceset="CPOL-EU" device="153CLV-0605" value="220uF"/>
-<part name="U$3" library="polargraph3" deviceset="MINI-360-MP2307" device=""/>
+<part name="U$3" library="polargraph3" deviceset="MINI-360-MP2307" device="MINI-360-MP2307_T" value="MINI-360-MP2307MINI-360-MP2307_T"/>
 <part name="C5" library="resistor" deviceset="C-EU" device="C0805" value="100nF"/>
 <part name="C6" library="resistor" deviceset="CPOL-EU" device="153CLV-0605" value="220uF"/>

Commit message: v3.1 changed servo supply voltage to 3.3v
Connections:
- net +3V3: now also SERVO.2
- net +5V: no longer SERVO.2
Other:
- note added: "ESP32"
- note added: "Encoder headers"
- note added: "Encoder voltage changers"
- note added: "LCD connector"
- note added: "Polarshield 3.1"
- note added: "Power"
- note added: "Servo"
- moved on the sheet: C1, C2, C7, C8, CN1, CN2, M1_CONN, M2_CONN, R2, R9, SJ1, SJ2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
